File: TFG-V1.kicad_pcb (KiCad board)
At the start: 2 copper layers, 50.9 x 74.4 mm, 69 parts, among them CN1 1n, CN2 1n, CN3 1n, CN4 1n, CN5 1n, J1 Input, U1 AMS1117-3.3, U10 TPS72325, U11 TPD4E1U06, U12 CRE1S0505SC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

Commit message: arreglo1
Parts:
- C15, C16, C22, C24, C34, C35, C7, C8, CN1, CN2, CN3, CN4, CN5, U11, U2, U4, U7, U8, U9: moved to F.Cu
- moved C15 38.1 mm to (153.0, 57.2), turned to 0 degrees
- moved C22 37.1 mm to (153.0, 55.2), turned to 0 degrees
- moved C7 36.6 mm to (153.0, 53.2), turned to 0 degrees
- moved C35 36.2 mm to (153.1, 51.2), turned to 0 degrees
- moved C16 33.1 mm to (153.3, 59.2)
- moved C8 27.6 mm to (153.2, 61.2)
- moved C6 15.5 mm to (153.0, 49.2), turned to 0 degrees
- moved U11 9.50 mm to (108.0, 49.8)
- moved U4 9.50 mm to (123.4, 49.6)
- moved U7 9.49 mm to (117.9, 49.7)
- moved U8 9.49 mm to (112.9, 49.7)
- moved U9 9.40 mm to (135.0, 49.6)
- moved J1 9.38 mm to (108.5, 45.8)
- moved U2 9.32 mm to (129.5, 49.7)
- moved C24 8.51 mm to (133.5, 70.7)
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Connections:
- CN1 pad 1: /IN_8P -> GNDD
- CN1 pad 2: /IN_8N -> GNDD
- CN1 pad 3: /IN_RLD_DRV -> GNDD
- CN1 pad 6: GNDD -> /IN_RLD_DRV
- CN1 pad 7: GNDD -> /IN_8N
- CN1 pad 8: GNDD -> /IN_8P
- CN2 pad 1: /IN_6P -> GNDD
- CN2 pad 2: /IN_6N -> GNDD
- CN2 pad 3: /IN_7P -> GNDD
- CN2 pad 4: /IN_7N -> GNDD
- CN2 pad 5: GNDD -> /IN_7N
- CN2 pad 6: GNDD -> /IN_7P
- CN2 pad 7: GNDD -> /IN_6N
- CN2 pad 8: GNDD -> /IN_6P
- CN3 pad 1: /IN_4P -> GNDD
- CN3 pad 2: /IN_4N -> GNDD
- CN3 pad 3: /IN_5P -> GNDD
- CN3 pad 4: /IN_5N -> GNDD
- CN3 pad 5: GNDD -> /IN_5N
- CN3 pad 6: GNDD -> /IN_5P
- CN3 pad 7: GNDD -> /IN_4N
- CN3 pad 8: GNDD -> /IN_4P
- CN4 pad 1: /IN_2P -> GNDD
- CN4 pad 2: /IN_2N -> GNDD
- CN4 pad 3: /IN_3P -> GNDD
- CN4 pad 4: /IN_3N -> GNDD
- CN4 pad 5: GNDD -> /IN_3N
- CN4 pad 6: GNDD -> /IN_3P
- CN4 pad 7: GNDD -> /IN_2N
- CN4 pad 8: GNDD -> /IN_2P
- CN5 pad 1: /IN_TESTP2 -> GNDD
- CN5 pad 2: /IN_TESTP1 -> GNDD
- CN5 pad 3: /IN_1P -> GNDD
- CN5 pad 4: /IN_1N -> GNDD
- CN5 pad 5: GNDD -> /IN_1N
- CN5 pad 6: GNDD -> /IN_1P
- CN5 pad 7: GNDD -> /IN_TESTP1
- CN5 pad 8: GNDD -> /IN_TESTP2
- RN1 pad 1: GNDD -> /IN_8P
- RN1 pad 2: /RLD_DRV -> /IN_8N
- RN1 pad 3: /8N -> /IN_RLD_DRV
- RN1 pad 4: /8P -> GNDD
- RN1 pad 5: /IN_8P -> GNDD
- RN1 pad 6: /IN_8N -> /RLD_DRV
- RN1 pad 7: /IN_RLD_DRV -> /8N
- RN1 pad 8: GNDD -> /8P
- RN2 pad 1: /7N -> /IN_6P
- RN2 pad 2: /7P -> /IN_6N
- RN2 pad 3: /6N -> /IN_7P
- RN2 pad 4: /6P -> /IN_7N
- RN2 pad 5: /IN_6P -> /7N
- RN2 pad 6: /IN_6N -> /7P
- RN2 pad 7: /IN_7P -> /6N
- RN2 pad 8: /IN_7N -> /6P
- RN3 pad 1: /5N -> /IN_4P
- RN3 pad 2: /5P -> /IN_4N
- RN3 pad 3: /4N -> /IN_5P
- RN3 pad 4: /4P -> /IN_5N
- RN3 pad 5: /IN_4P -> /5N
- RN3 pad 6: /IN_4N -> /5P
- RN3 pad 7: /IN_5P -> /4N
- RN3 pad 8: /IN_5N -> /4P
- RN4 pad 1: /3N -> /IN_2P
- RN4 pad 2: /3P -> /IN_2N
- RN4 pad 3: /2N -> /IN_3P
- RN4 pad 4: /2P -> /IN_3N
- RN4 pad 5: /IN_2P -> /3N
- RN4 pad 6: /IN_2N -> /3P
- RN4 pad 7: /IN_3P -> /2N
- RN4 pad 8: /IN_3N -> /2P
- RN5 pad 1: /1N -> /IN_TESTP2
- RN5 pad 2: /1P -> /IN_TESTP1
- RN5 pad 3: /TESTP1 -> /IN_1P
- RN5 pad 4: /TESTP2 -> /IN_1N
- RN5 pad 5: /IN_TESTP2 -> /1N
- RN5 pad 6: /IN_TESTP1 -> /1P
- RN5 pad 7: /IN_1P -> /TESTP1
- RN5 pad 8: /IN_1N -> /TESTP2
Routing:
- net GNDD: track 237.2 -> 276.5 mm, vias 20 -> 17
- net GND: track 133.4 -> 159.0 mm, vias 3 -> 0
- net VDDA: track 104.1 -> 128.6 mm, vias 8 -> 2
- net Net-(U3-WCT): track 3.59 -> 27.9 mm, vias 1 -> 2
- net VSSA: track 124.5 -> 146.2 mm, vias 7 -> 10
- net /5V_ISO: track 73.9 -> 91.8 mm, vias 0 -> 4
- net VDD: track 76.2 -> 91.0 mm, vias 2 -> 6
- net /6N: track 4.70 -> 13.6 mm, vias 1 -> 0
- net /8N: track 5.99 -> 12.3 mm
- net /2N: track 6.09 -> 12.3 mm
- net /4N: track 6.18 -> 12.3 mm
- net +5V: track 54.0 -> 60.1 mm, vias 1 -> 2
- net /IN_7P: track 7.90 -> 13.9 mm, vias 1 -> 0
- net /FE_START_ISO: track 5.78 -> 11.7 mm
- net /IN_5P: track 6.83 -> 12.6 mm, vias 1 -> 0
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- removed copper zone on F.Cu, net +5V
- removed copper zone on F.Cu, net VSSA
Other:
- board size 50.9 x 74.4 mm -> 55 x 90 mm

Commit message: correcciones varias 1
reruteo y corregir algunas cosas
Parts:
- moved C15 47.5 mm to (107.0, 69.2), turned to 180 degrees
- moved C35 47.2 mm to (115.0, 79.2), turned to 180 degrees
- moved C32 45.4 mm to (147.4, 51.8), turned to 90 degrees
- moved C23 43.4 mm to (107.0, 74.3), turned to 180 degrees
- moved C22 43.1 mm to (111.5, 66.5), turned to 180 degrees
- moved C12 39.3 mm to (144.4, 69.3), turned to -90 degrees
- moved C1 37.1 mm to (141.4, 82.8), turned to -90 degrees
- moved C2 35.4 mm to (138.4, 82.8), turned to -90 degrees
- moved C4 34.9 mm to (107.0, 79.5), turned to 180 degrees
- moved C3 32.0 mm to (107.0, 77.0), turned to 180 degrees
- moved C38 29.3 mm to (115.0, 81.8)
- moved C6 27.1 mm to (141.4, 73.8), turned to 90 degrees
- moved C7 22.2 mm to (144.4, 73.8), turned to 90 degrees
- moved C8 21.1 mm to (132.1, 62.1)
- moved U6 20.9 mm to (150.2, 73.3), turned to 0 degrees
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Connections:
- D3 pad 1: Net-(D3-K) -> GNDD
- D3 pad 2: VDD -> Net-(D3-A)
- R1 pad 1: GNDD -> Net-(D3-A)
- R1 pad 2: Net-(D3-K) -> VDD
- U11 pad 1: /TESTP2 -> VSSA
- U11 pad 3: VSSA -> /TESTP2
- U2 pad 1: /7P -> /7N
- U2 pad 3: /7N -> /7P
- U4 pad 1: /5P -> /5N
- U4 pad 3: /5N -> /5P
- U7 pad 1: /3P -> /3N
- U7 pad 3: /3N -> /3P
- U8 pad 1: /1P -> /1N
- U8 pad 3: /1N -> /1P
Routing:
- net GNDD: track 276.5 -> 136.5 mm, vias 17 -> 37
- net /5V_ISO: track 91.8 -> 16.7 mm, vias 4 -> 0
- net VDDA: track 128.6 -> 106.1 mm, vias 2 -> 5
- net Net-(U3-WCT): track 27.9 -> 7.60 mm, vias 2 -> 0
- net /Vneg_raw: track 7.05 -> 22.2 mm
- net +5V: track 60.1 -> 46.1 mm
- net GND: track 159.0 -> 147.5 mm
- net Net-(U3-VREFP): track 25.7 -> 15.5 mm
- net /VCAP4: track 9.26 -> 3.27 mm, vias 2 -> 0
- net Net-(U5-CAP+): track 5.38 -> 9.88 mm
- net /7N: track 9.11 -> 13.1 mm
- net /2N: track 12.3 -> 8.45 mm
- net /5N: track 8.10 -> 11.7 mm
- net /3P: track 11.0 -> 14.6 mm
- net /RLD_DRV: track 12.7 -> 16.2 mm
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
Commit message: diseño final
Parts:
- J1: footprint Connector_PinHeader_2.54mm:PinHeader_2x13_P2.54mm_Horizontal -> Connector_PinHeader_2.54mm:PinHeader_2x13_P2.54mm_Vertical
- moved BT1 10.1 mm to (151.0, 89.5), turned to 0 degrees
- moved U14 2.18 mm to (112.8, 118.5)
- moved C34 1.55 mm to (142.2, 88.3)
- moved U1 1.25 mm to (149.0, 81.1)
- moved D1 0.75 mm to (138.8, 88.8)
- moved U15 0.50 mm to (121.8, 86.5)
- moved C38 0.45 mm to (115.0, 82.3)
Routing:
- net GND: track 147.5 -> 24.9 mm
- net /FE_CS: track 7.62 -> 16.9 mm
- net /BAT_IN: track 19.5 -> 13.8 mm
- net 3V3: track 37.4 -> 41.7 mm
- net /SPI1_SCLK: track 32.4 -> 36.6 mm
- net /FE_DRDY: track 14.8 -> 11.1 mm
- net /SPI1_MISO: track 7.93 -> 6.08 mm, vias 2 -> 0
- net /SPI1_MOSI: track 33.1 -> 34.9 mm
- net +5V: track 46.1 -> 47.8 mm
- net VDD: track 90.3 -> 88.8 mm
- net /5V_ISO: track 16.7 -> 15.5 mm
- net /FE_START: track 6.77 -> 5.72 mm, vias 2 -> 0
- net /FE_RESET: track 13.3 -> 12.5 mm
- net /SPI1_SCLK_ISO: track 7.35 -> 6.85 mm
- net /SPI1_MOSI_ISO: track 11.6 -> 11.1 mm
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- added copper zone on F.Cu, net GND
- added copper zone on F.Cu, net GNDD
Other:
- board size 55 x 90 mm -> 50 x 80 mm
