File: TFG-V1.kicad_sch (KiCad schematic)
At the start: 69 parts, among them CN1 1n, CN2 1n, CN3 1n, CN4 1n, CN5 1n, J1 Input, U1 AMS1117-3.3, U10 TPS72325, U11 TPD4E1U06, U12 CRE1S0505SC, U14 ESP32-C3-DevKitC-02, U15 ADuM3151, U2 TPD4E1U06, U3 ADS1298PAG, U4 TPD4E1U06, U5 LM2664, U6 MIC5504-2.5YM5, U7 TPD4E1U06, U8 TPD4E1U06, U9 TPD4E1U06

Commit message: arreglo1
Connections:
- net 1N: now also RN5.5 (R4.2); no longer RN5.1 (R1.1)
- net 1P: now also RN5.6 (R3.2); no longer RN5.2 (R2.1)
- net 2N: now also RN4.7 (R2.2); no longer RN4.3 (R3.1)
- net 2P: now also RN4.8 (R1.2); no longer RN4.4 (R4.1)
- net 3N: now also RN4.5 (R4.2); no longer RN4.1 (R1.1)
- net 3P: now also RN4.6 (R3.2); no longer RN4.2 (R2.1)
- net 4N: now also RN3.7 (R2.2); no longer RN3.3 (R3.1)
- net 4P: now also RN3.8 (R1.2); no longer RN3.4 (R4.1)
- net 5N: now also RN3.5 (R4.2); no longer RN3.1 (R1.1)
- net 5P: now also RN3.6 (R3.2); no longer RN3.2 (R2.1)
- net 6N: now also RN2.7 (R2.2); no longer RN2.3 (R3.1)
- net 6P: now also RN2.8 (R1.2); no longer RN2.4 (R4.1)
- net 7N: now also RN2.5 (R4.2); no longer RN2.1 (R1.1)
- net 7P: now also RN2.6 (R3.2); no longer RN2.2 (R2.1)
- net 8N: now also RN1.7 (R2.2); no longer RN1.3 (R3.1)
- net 8P: now also RN1.8 (R1.2); no longer RN1.4 (R4.1)
- net GNDD: now also CN1.1 (R1.1), CN1.2 (R2.1), CN1.3 (R3.1), CN2.1 (R1.1), CN2.2 (R2.1), CN2.3 (R3.1), CN2.4 (R4.1), CN3.1 (R1.1), CN3.2 (R2.1), CN3.3 (R3.1), CN3.4 (R4.1), CN4.1 (R1.1), CN4.2 (R2.1), CN4.3 (R3.1), CN4.4 (R4.1), CN5.1 (R1.1), CN5.2 (R2.1), CN5.3 (R3.1), CN5.4 (R4.1), RN1.4 (R4.1), RN1.5 (R4.2); no longer CN1.6 (R3.2), CN1.7 (R2.2), CN1.8 (R1.2), CN2.5 (R4.2), CN2.6 (R3.2), CN2.7 (R2.2), CN2.8 (R1.2), CN3.5 (R4.2), CN3.6 (R3.2), CN3.7 (R2.2), CN3.8 (R1.2), CN4.5 (R4.2), CN4.6 (R3.2), CN4.7 (R2.2), CN4.8 (R1.2), CN5.5 (R4.2), CN5.6 (R3.2), CN5.7 (R2.2), CN5.8 (R1.2), RN1.1 (R1.1), RN1.8 (R1.2)
- net IN_1N: now also CN5.5 (R4.2), RN5.4 (R4.1); no longer CN5.4 (R4.1), RN5.8 (R1.2)
- net IN_1P: now also CN5.6 (R3.2), RN5.3 (R3.1); no longer CN5.3 (R3.1), RN5.7 (R2.2)
- net IN_2N: now also CN4.7 (R2.2), RN4.2 (R2.1); no longer CN4.2 (R2.1), RN4.6 (R3.2)
- net IN_2P: now also CN4.8 (R1.2), RN4.1 (R1.1); no longer CN4.1 (R1.1), RN4.5 (R4.2)
- net IN_3N: now also CN4.5 (R4.2), RN4.4 (R4.1); no longer CN4.4 (R4.1), RN4.8 (R1.2)
- net IN_3P: now also CN4.6 (R3.2), RN4.3 (R3.1); no longer CN4.3 (R3.1), RN4.7 (R2.2)
- net IN_4N: now also CN3.7 (R2.2), RN3.2 (R2.1); no longer CN3.2 (R2.1), RN3.6 (R3.2)
- net IN_4P: now also CN3.8 (R1.2), RN3.1 (R1.1); no longer CN3.1 (R1.1), RN3.5 (R4.2)
- net IN_5N: now also CN3.5 (R4.2), RN3.4 (R4.1); no longer CN3.4 (R4.1), RN3.8 (R1.2)
- net IN_5P: now also CN3.6 (R3.2), RN3.3 (R3.1); no longer CN3.3 (R3.1), RN3.7 (R2.2)
- net IN_6N: now also CN2.7 (R2.2), RN2.2 (R2.1); no longer CN2.2 (R2.1), RN2.6 (R3.2)
- net IN_6P: now also CN2.8 (R1.2), RN2.1 (R1.1); no longer CN2.1 (R1.1), RN2.5 (R4.2)
- net IN_7N: now also CN2.5 (R4.2), RN2.4 (R4.1); no longer CN2.4 (R4.1), RN2.8 (R1.2)
- net IN_7P: now also CN2.6 (R3.2), RN2.3 (R3.1); no longer CN2.3 (R3.1), RN2.7 (R2.2)
- net IN_8N: now also CN1.7 (R2.2), RN1.2 (R2.1); no longer CN1.2 (R2.1), RN1.6 (R3.2)
- net IN_8P: now also CN1.8 (R1.2), RN1.1 (R1.1); no longer CN1.1 (R1.1), RN1.5 (R4.2)
- net IN_RLD_DRV: now also CN1.6 (R3.2), RN1.3 (R3.1); no longer CN1.3 (R3.1), RN1.7 (R2.2)
- net IN_TESTP1: now also CN5.7 (R2.2), RN5.2 (R2.1); no longer CN5.2 (R2.1), RN5.6 (R3.2)
- net IN_TESTP2: now also CN5.8 (R1.2), RN5.1 (R1.1); no longer CN5.1 (R1.1), RN5.5 (R4.2)
- net RLD_DRV: now also RN1.6 (R3.2); no longer RN1.2 (R2.1)
- net TESTP1: now also RN5.7 (R2.2); no longer RN5.3 (R3.1)
- net TESTP2: now also RN5.8 (R1.2); no longer RN5.4 (R4.1)
Other:
- moved on the sheet: CN1, CN2, CN3, CN4, CN5, RN1, RN2, RN3, RN4, RN5
Changed lines of the file:
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@@
 	)
 	(junction
-		(at 364.49 196.85)
-		(diameter 0)
-		(color 0 0 0 0)
-	)
-	(junction
 		(at 234.95 259.08)
 		(diameter 0)
@@
 	)
 	(junction
+		(at 364.49 196.85)
+		(diameter 0)
+		(color 0 0 0 0)
+	)
+	(junction
 		(at 262.89 196.85)
 		(diameter 0)
@@
 	(symbol
 		(lib_id "C10418:C_Pack04")
-		(at 290.83 191.77 180)
+		(at 290.83 191.77 0)
+		(mirror y)
 		(unit 1)
 		(exclude_from_sim no)
@@
 		(dnp no)
 		(property "Reference" "CN3"
-			(at 297.942 190.6016 0)
+			(at 297.942 192.9384 0)
 			(effects
 				(font
@@
 		)
 		(property "Value" "1n"
-			(at 297.942 192.913 0)
+			(at 297.942 190.627 0)
 			(effects
 				(font
@@
 	(symbol
 		(lib_id "Device:R_Pack04")
-		(at 314.96 182.88 270)
+		(at 314.96 180.34 90)
 		(unit 1)
 		(exclude_from_sim no)
@@
 		(dnp no)
 		(property "Reference" "RN4"
-			(at 314.96 172.2882 90)
+			(at 314.96 190.9318 90)
 			(effects
 				(font
@@
 		)
 		(property "Value" "2.2k"
-			(at 314.96 174.5996 90)
+			(at 314.96 188.6204 90)
 			(effects
 				(font
@@
 		)
 		(property "Footprint" "Resistor_SMD:R_Array_Convex_4x0603"
-			(at 314.96 189.865 90)
+			(at 314.96 173.355 90)
 			(effects
 				(font
@@
 		)
 		(property "Datasheet" "~"
-			(at 314.96 182.88 0)
+			(at 314.96 180.34 0)
 			(effects
 				(font
@@
 		)
 		(property "Description" ""
-			(at 314.96 182.88 0)
+			(at 314.96 180.34 0)
 			(effects
 				(font
@@
 		)
 		(property "LCSC" "C12001"
-			(at 314.96 182.88 0)
+			(at 314.96 180.34 0)
 			(effects
 				(font
@@
 	(symbol
 		(lib_id "Device:R_Pack04")
-		(at 281.94 182.88 270)
+		(at 281.94 180.34 90)
 		(unit 1)
 		(exclude_from_sim no)
@@
 		(dnp no)
 		(property "Reference" "RN3"
-			(at 281.94 172.2882 90)
+			(at 281.94 190.9318 90)
 			(effects
 				(font
@@
 		)
 		(property "Value" "2.2k"
-			(at 281.94 174.5996 90)
+			(at 281.94 188.6204 90)
 			(effects
 				(font
@@
 		)
 		(property "Footprint" "Resistor_SMD:R_Array_Convex_4x0603"
-			(at 281.94 189.865 90)
+			(at 281.94 173.355 90)
 			(effects
 				(font
@@
 		)
 		(property "Datasheet" "~"
-			(at 281.94 182.88 0)
+			(at 281.94 180.34 0)
 			(effects
 				(font
@@
 		)
 		(property "Description" ""
-			(at 281.94 182.88 0)
+			(at 281.94 180.34 0)
 			(effects
 				(font
@@
 		)
 		(property "LCSC" "C12001"
-			(at 281.94 182.88 0)
+			(at 281.94 180.34 0)
 			(effects
 				(font
@@
 	(symbol
 		(lib_id "Device:R_Pack04")
-		(at 248.92 182.88 270)
+		(at 248.92 180.34 90)
 		(unit 1)
 		(exclude_from_sim no)
@@
 		(dnp no)
 		(property "Reference" "RN2"
-			(at 248.92 172.2882 90)
+			(at 248.92 190.9318 90)
 			(effects
 				(font
@@
 		)
 		(property "Value" "2.2k"
-			(at 248.92 174.5996 90)
+			(at 248.92 188.6204 90)
 			(effects
 				(font
@@
 		)
 		(property "Footprint" "Resistor_SMD:R_Array_Convex_4x0603"
-			(at 248.92 189.865 90)
+			(at 248.92 173.355 90)
 			(effects
 				(font
@@
 		)
 		(property "Datasheet" "~"
-			(at 248.92 182.88 0)
+			(at 248.92 180.34 0)
 			(effects
 				(font
@@
 		)
 		(property "Description" ""
-			(at 248.92 182.88 0)
+			(at 248.92 180.34 0)
 			(effects
 				(font
@@
 		)
 		(property "LCSC" "C12001"
-			(at 248.92 182.88 0)
+			(at 248.92 180.34 0)
 			(effects
 				(font
@@
 		(on_board yes)
 		(dnp no)
-		(fields_autoplaced yes)
 		(property "Reference" "U15"
 			(at 152.0541 73.66 0)
@@
 	(symbol
 		(lib_id "C10418:C_Pack04")
-		(at 257.81 191.77 180)
+		(at 257.81 191.77 0)
+		(mirror y)
 		(unit 1)
 		(exclude_from_sim no)
@@
 		(dnp no)
 		(property "Reference" "CN2"
-			(at 264.922 190.6016 0)
+			(at 264.922 192.9384 0)
 			(effects
 				(font
@@
 		)
 		(property "Value" "1n"
-			(at 264.922 192.913 0)
+			(at 264.922 190.627 0)
 			(effects
 				(font
@@
 	(symbol
 		(lib_id "Device:R_Pack04")
-		(at 215.9 182.88 270)
+		(at 215.9 180.34 90)
 		(unit 1)
 		(exclude_from_sim no)
@@
 		(dnp no)
 		(property "Reference" "RN1"
-			(at 215.9 172.2882 90)
+			(at 215.9 190.9318 90)
 			(effects
 				(font
@@
 		)
 		(property "Value" "2.2k"
-			(at 215.9 174.5996 90)
+			(at 215.9 188.6204 90)
 			(effects
 				(font
@@
 		)
 		(property "Footprint" "Resistor_SMD:R_Array_Convex_4x0603"
-			(at 215.9 189.865 90)
+			(at 215.9 173.355 90)
 			(effects
 				(font
@@
 		)
 		(property "Datasheet" "~"
-			(at 215.9 182.88 0)
+			(at 215.9 180.34 0)
 			(effects
 				(font
@@
 		)
 		(property "Description" ""
-			(at 215.9 182.88 0)
+			(at 215.9 180.34 0)
 			(effects
 				(font
@@
 		)
 		(property "LCSC" "C12001"
-			(at 215.9 182.88 0)
+			(at 215.9 180.34 0)
 			(effects
 				(font
@@
 	(symbol
 		(lib_id "C10418:C_Pack04")
-		(at 323.85 191.77 180)
+		(at 323.85 191.77 0)
+		(mirror y)
 		(unit 1)
 		(exclude_from_sim no)
@@
 		(dnp no)
 		(property "Reference" "CN4"
-			(at 330.962 190.6016 0)
+			(at 330.962 192.9384 0)
 			(effects
 				(font
@@
 		)
 		(property "Value" "1n"
-			(at 330.962 192.913 0)
+			(at 330.962 190.627 0)
 			(effects
 				(font
@@
 	(symbol
 		(lib_id "C10418:C_Pack04")
-		(at 359.41 191.77 180)
+		(at 359.41 191.77 0)
+		(mirror y)
 		(unit 1)
 		(exclude_from_sim no)
@@
 		(dnp no)
 		(property "Reference" "CN5"
-			(at 366.522 190.6016 0)
+			(at 366.522 192.9384 0)
 			(effects
 				(font
@@
 		)
 		(property "Value" "1n"
-			(at 366.522 192.913 0)
+			(at 366.522 190.627 0)
 			(effects
 				(font
@@
 	(symbol
 		(lib_id "C10418:C_Pack04")
-		(at 224.79 191.77 180)
+		(at 224.79 191.77 0)
+		(mirror y)
 		(unit 1)
 		(exclude_from_sim no)
@@
 		(dnp no)
 		(property "Reference" "CN1"
-			(at 231.902 190.6016 0)
+			(at 231.902 192.9384 0)
 			(effects
 				(font
@@
 		)
 		(property "Value" "1n"
-			(at 231.902 192.913 0)
+			(at 231.902 190.627 0)
 			(effects
 				(font
@@
 	(symbol
 		(lib_id "Device:R_Pack04")
-		(at 350.52 182.88 270)
+		(at 350.52 180.34 90)
 		(unit 1)
 		(exclude_from_sim no)
@@
 		(dnp no)
 		(property "Reference" "RN5"
-			(at 350.52 172.2882 90)
+			(at 350.52 190.9318 90)
 			(effects
 				(font
@@
 		)
 		(property "Value" "2.2k"
-			(at 350.52 174.5996 90)
+			(at 350.52 188.6204 90)
 			(effects
 				(font
@@
 		)
 		(property "Footprint" "Resistor_SMD:R_Array_Convex_4x0603"
-			(at 350.52 189.865 90)
+			(at 350.52 173.355 90)
 			(effects
 				(font
@@
 		)
 		(property "Datasheet" "~"
-			(at 350.52 182.88 0)
+			(at 350.52 180.34 0)
 			(effects
 				(font
@@
 		)
 		(property "Description" ""
-			(at 350.52 182.88 0)
+			(at 350.52 180.34 0)
 			(effects
 				(font
@@
 		)
 		(property "LCSC" "C12001"
-			(at 350.52 182.88 0)
+			(at 350.52 180.34 0)
 			(effects
 				(font

Commit message: correcciones varias 1
reruteo y corregir algunas cosas
Connections:
- net 1N: now also U8.1 (D1+); no longer U8.3 (D2+)
- net 1P: now also U8.3 (D2+); no longer U8.1 (D1+)
- net 3N: now also U7.1 (D1+); no longer U7.3 (D2+)
- net 3P: now also U7.3 (D2+); no longer U7.1 (D1+)
- net 5N: now also U4.1 (D1+); no longer U4.3 (D2+)
- net 5P: now also U4.3 (D2+); no longer U4.1 (D1+)
- net 7N: now also U2.1 (D1+); no longer U2.3 (D2+)
- net 7P: now also U2.3 (D2+); no longer U2.1 (D1+)
- net GNDD: now also D3.1 (K); no longer R1.1
- net TESTP2: now also U11.3 (D2+); no longer U11.1 (D1+)
- net VDD: now also R1.2; no longer D3.2 (A)
- net VSSA: now also U11.1 (D1+); no longer U11.3 (D2+)
- new net: D3.2 (A), R1.1
Other:
- moved on the sheet: D3, R1, U11
Changed lines of the file:
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@@
 	)
 	(junction
-		(at 67.31 262.89)
-		(diameter 0)
-		(color 0 0 0 0)
-	)
-	(junction
 		(at 364.49 185.42)
 		(diameter 0)
@@
 	)
 	(junction
+		(at 67.31 262.89)
+		(diameter 0)
+		(color 0 0 0 0)
+	)
+	(junction
 		(at 33.02 262.89)
 		(diameter 0)
@@
 	)
 	(no_connect
-		(at 382.27 213.36)
+		(at 389.89 213.36)
 	)
 	(no_connect
@@
 	(wire
 		(pts
+			(xy 363.22 207.01) (xy 363.22 213.36)
+		)
+		(stroke
+			(width 0)
+			(type default)
+		)
+	)
+	(wire
+		(pts
 			(xy 218.44 78.74) (xy 207.01 78.74)
 		)
@@
 	(wire
 		(pts
+			(xy 363.22 213.36) (xy 369.57 213.36)
+		)
+		(stroke
+			(width 0)
+			(type default)
+		)
+	)
+	(wire
+		(pts
 			(xy 256.54 73.66) (xy 259.08 73.66)
 		)
@@
 	(wire
 		(pts
-			(xy 358.14 218.44) (xy 361.95 218.44)
+			(xy 365.76 218.44) (xy 369.57 218.44)
 		)
 		(stroke
@@
 	(wire
 		(pts
-			(xy 358.14 213.36) (xy 361.95 213.36)
+			(xy 367.03 207.01) (xy 363.22 207.01)
 		)
 		(stroke
@@
 	(wire
 		(pts
-			(xy 382.27 218.44) (xy 386.08 218.44)
+			(xy 389.89 218.44) (xy 393.7 218.44)
 		)
 		(stroke
@@
 	)
 	(label "7N"
-		(at 205.74 218.44 0)
+		(at 205.74 213.36 0)
 		(fields_autoplaced yes)
 		(effects
@@
 	)
 	(label "1P"
-		(at 298.45 213.36 0)
+		(at 298.45 218.44 0)
 		(fields_autoplaced yes)
 		(effects
@@
 	)
 	(label "5N"
-		(at 237.49 218.44 0)
+		(at 237.49 213.36 0)
 		(fields_autoplaced yes)
 		(effects
@@
 	)
 	(label "3P"
-		(at 267.97 213.36 0)
+		(at 267.97 218.44 0)
 		(fields_autoplaced yes)
 		(effects
@@
 	)
 	(label "TESTP1"
-		(at 386.08 218.44 0)
+		(at 393.7 218.44 0)
 		(fields_autoplaced yes)
 		(effects
@@
 	)
 	(label "5P"
-		(at 237.49 213.36 0)
+		(at 237.49 218.44 0)
 		(fields_autoplaced yes)
 		(effects
@@
 	)
 	(label "1N"
-		(at 298.45 218.44 0)
+		(at 298.45 213.36 0)
 		(fields_autoplaced yes)
 		(effects
@@
 	)
 	(label "TESTP2"
-		(at 358.14 213.36 0)
+		(at 365.76 218.44 180)
 		(fields_autoplaced yes)
 		(effects
@@
 				(size 1.27 1.27)
 			)
-			(justify left bottom)
+			(justify right bottom)
 		)
 	)
@@
 	)
 	(label "3N"
-		(at 267.97 218.44 0)
+		(at 267.97 213.36 0)
 		(fields_autoplaced yes)
 		(effects
@@
 	)
 	(label "7P"
-		(at 205.74 213.36 0)
+		(at 205.74 218.44 0)
 		(fields_autoplaced yes)
 		(effects
@@
 	(symbol
 		(lib_id "C10418:TPD4E1U06")
-		(at 372.11 214.63 0)
+		(at 379.73 214.63 0)
 		(unit 1)
 		(exclude_from_sim no)
@@
 		(dnp no)
 		(property "Reference" "U11"
-			(at 372.11 208.28 0)
+			(at 379.73 208.28 0)
 			(effects
 				(font
@@
 		)
 		(property "Value" "TPD4E1U06"
-			(at 372.11 210.82 0)
+			(at 379.73 210.82 0)
 			(effects
 				(font
@@
 		)
 		(property "Footprint" "Package_TO_SOT_SMD:SOT-23-6"
-			(at 372.11 218.44 0)
+			(at 379.73 218.44 0)
 			(effects
 				(font
@@
 		)
 		(property "Datasheet" ""
-			(at 372.11 215.9 0)
+			(at 379.73 215.9 0)
 			(effects
 				(font
@@
 		)
 		(property "Description" ""
-			(at 372.11 214.63 0)
+			(at 379.73 214.63 0)
 			(effects
 				(font
@@
 		)
 		(property "LCSC" "C124691"
-			(at 372.11 214.63 0)
+			(at 379.73 214.63 0)
 			(effects
 				(font
@@
 		)
 		(property "Value" "VDDA"
-			(at 353.4918 214.0458 0)
+			(at 353.568 220.218 0)
 			(effects
 				(font
@@
 	(symbol
 		(lib_id "Device:LED")
-		(at 71.12 262.89 180)
+		(at 74.93 266.7 90)
 		(unit 1)
 		(exclude_from_sim no)
@@
 		(dnp no)
 		(property "Reference" "D3"
-			(at 70.1294 259.9182 90)
+			(at 77.9018 265.7094 90)
 			(effects
 				(font
@@
 		)
 		(property "Value" "PWR_LED"
-			(at 72.4408 259.9182 90)
+			(at 77.9018 268.0208 90)
 			(effects
 				(font
@@
 		)
 		(property "Footprint" "LED_SMD:LED_0805_2012Metric"
-			(at 71.12 262.89 0)
+			(at 74.93 266.7 0)
 			(effects
 				(font
@@
 		)
 		(property "Datasheet" "~"
-			(at 71.12 262.89 0)
+			(at 74.93 266.7 0)
 			(effects
 				(font
@@
 		)
 		(property "Description" ""
-			(at 71.12 262.89 0)
+			(at 74.93 266.7 0)
 			(effects
 				(font
@@
 		)
 		(property "LCSC" "C72037"
-			(at 71.12 262.89 0)
+			(at 74.93 266.7 0)
 			(effects
 				(font
@@
 	(symbol
 		(lib_id "power:GNDD")
-		(at 372.11 222.25 0)
+		(at 379.73 222.25 0)
 		(unit 1)
 		(exclude_from_sim no)
@@
 		(dnp no)
 		(property "Reference" "#PWR064"
-			(at 372.11 228.6 0)
+			(at 379.73 228.6 0)
 			(effects
 				(font
@@
 		)
 		(property "Value" "GNDD"
-			(at 372.2116 226.187 0)
+			(at 379.8316 226.187 0)
 			(effects
 				(font
@@
 		)
 		(property "Footprint" ""
-			(at 372.11 222.25 0)
+			(at 379.73 222.25 0)
 			(effects
 				(font
@@
 		)
 		(property "Datasheet" ""
-			(at 372.11 222.25 0)
+			(at 379.73 222.25 0)
 			(effects
 				(font
@@
 		)
 		(property "Description" ""
-			(at 372.11 222.25 0)
+			(at 379.73 222.25 0)
 			(effects
 				(font
@@
 		)
 		(instances
-			(project ""
+			(project "TFG-V1"
 				(path "/abf25f1f-efb8-4985-80da-541cd4215f12"
 					(reference "U15")
@@
 		)
 		(instances
-			(project ""
+			(project "TFG-V1"
 				(path "/abf25f1f-efb8-4985-80da-541cd4215f12"
 					(reference "U14")
@@
 	(symbol
 		(lib_id "Device:R")
-		(at 74.93 266.7 180)
+		(at 71.12 262.89 270)
 		(unit 1)
 		(exclude_from_sim no)
@@
 		(dnp no)
 		(property "Reference" "R1"
-			(at 72.39 266.7 90)
+			(at 71.12 265.43 90)
 			(effects
 				(font
@@
 		)
 		(property "Value" "1k"
-			(at 74.93 266.7 90)
+			(at 71.12 262.89 90)
 			(effects
 				(font
@@
 		)
 		(property "Footprint" "Resistor_SMD:R_0805_2012Metric"
-			(at 76.708 266.7 90)
+			(at 71.12 261.112 90)
 			(effects
 				(font
@@
 		)
 		(property "Datasheet" "~"
-			(at 74.93 266.7 0)
+			(at 71.12 262.89 0)
 			(effects
 				(font
@@
 		)
 		(property "Description" ""
-			(at 74.93 266.7 0)
+			(at 71.12 262.89 0)
 			(effects
 				(font
@@
 		)
 		(property "LCSC" "C17513"
-			(at 74.93 266.7 0)
+			(at 71.12 262.89 0)
 			(effects
 				(font
@@
 	(symbol
 		(lib_id "power:VSSA")
-		(at 358.14 218.44 180)
+		(at 367.03 207.01 180)
 		(unit 1)
 		(exclude_from_sim no)
@@
 		(dnp no)
 		(property "Reference" "#PWR060"
-			(at 358.14 214.63 0)
+			(at 367.03 203.2 0)
 			(effects
 				(font
@@
 		)
 		(property "Value" "VSSA"
-			(at 357.6828 222.8342 0)
+			(at 366.5728 211.4042 0)
 			(effects
 				(font
@@
 		)
 		(property "Footprint" ""
-			(at 358.14 218.44 0)
+			(at 367.03 207.01 0)
 			(effects
 				(font
@@
 		)
 		(property "Datasheet" ""
-			(at 358.14 218.44 0)
+			(at 367.03 207.01 0)
 			(effects
 				(font
@@
 		)
 		(property "Description" ""
-			(at 358.14 218.44 0)
+			(at 367.03 207.01 0)
 			(effects
 				(font
@@
 		)
 		(instances
-			(project ""
+			(project "TFG-V1"
 				(path "/abf25f1f-efb8-4985-80da-541cd4215f12"
 					(reference "U6")

Commit message: diseño final
Parts:
- J1: footprint Connector_PinHeader_2.54mm:PinHeader_2x13_P2.54mm_Horizontal -> Connector_PinHeader_2.54mm:PinHeader_2x13_P2.54mm_Vertical
Changed lines of the file:
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@@
 			)
 		)
-		(property "Footprint" "Connector_PinHeader_2.54mm:PinHeader_2x13_P2.54mm_Horizontal"
+		(property "Footprint" "Connector_PinHeader_2.54mm:PinHeader_2x13_P2.54mm_Vertical"
 			(at 383.54 67.31 0)
 			(effects
